File: LQFP48-Breakout.kicad_pcb (KiCad board)
At the start: 2 copper layers, 20.3 x 63.5 mm, 2 parts, among them J1 Conn_02x24_Counter_Clockwise, U1 NUC029LAN

Commit message: migrate to v6
Other:
- net class Default removed
